File: moduloSonido/moduloSonidoPCB/moduloSonidoPCB.kicad_pcb (KiCad board)
At the start: 2 copper layers, 25.4 x 34.3 mm, 8 parts, among them J1 Conn_01x03, J2 Conn_01x05, U1 ATtiny85V-10P

Commit message: PCB 1.1
Capacitor y plano de tierra agregados
Parts:
- removed REF** (x2): MountingHole_2.5mm_Pad, MountingHole:MountingHole_2.5mm_Pad
- added C1: 10u, Capacitor_THT:CP_Radial_D5.0mm_P2.50mm, F.Cu at (100.9, 49.2)
- added REF1: MountingHole_2.5mm, MountingHole:MountingHole_2.5mm, F.Cu at (109.6, 50.2)
- added REF2: MountingHole_2.5mm, MountingHole:MountingHole_2.5mm, F.Cu at (91.1, 50.2)
- added REF3: MountingHole_2.5mm, MountingHole:MountingHole_2.5mm, F.Cu at (110.1, 20.8)
- added REF4: MountingHole_2.5mm, MountingHole:MountingHole_2.5mm, F.Cu at (90.8, 20.8)
- moved D1 13.3 mm to (93.9, 40.1)
- moved J1 13.3 mm to (103.4, 21.0)
- moved J2 13.3 mm to (107.2, 40.1)
- moved R1 13.3 mm to (104.7, 44.5)
- moved R2 13.3 mm to (95.8, 25.5)
- moved U1 13.3 mm to (97.0, 28.7)
Routing:
- net +3V3: track 21.7 -> 34.4 mm
- net GND: track 29.9 -> 38.3 mm
- added copper zone on F.Cu, net GND
Other:
- board size 25.4 x 34.3 mm -> 25.4 x 33.8 mm

Commit message: Actualizacion PCB
Algunos cambios en diseño de PCB
Parts:
- moved C1 64.4 mm to (129.7, 106.8)
- moved R1 64.4 mm to (133.5, 102.1)
- moved R2 64.4 mm to (124.6, 83.1)
- moved D1 64.4 mm to (122.7, 97.7)
- moved J1 64.4 mm to (132.2, 78.6)
- moved J2 64.4 mm to (136.0, 97.7)
- moved REF1 64.4 mm to (138.4, 107.8)
- moved REF2 64.4 mm to (119.9, 107.8)
- moved REF3 64.4 mm to (138.9, 78.4)
- moved REF4 64.4 mm to (119.6, 78.4)
- moved U1 64.4 mm to (125.8, 86.2)
