File: placaConexiones/placa/placa.kicad_sch (KiCad schematic)
At the start: 8 parts, among them J1 Conn_01x05, J2 Conn_01x05, J3 Conn_01x06, J4 Conn_01x09

Commit message: Actualizacion esquematico de placa
Other:
- note added: "1.0"
- note added: "18/02/2022"
- note added: "3.3V"
- note added: "F"
- note added: "GPS B"
- note added: "GPS T"
- note added: "NOTA: Verificar la impresión"
- note added: "Placa para conexiones"
- note added: "SM300 F"
- note added: "SM300 TD"
- note added: "SONIDO F"
- note added: "SONIDO Tx"
- note added: "ailr16"
- note removed: "Dig"
- moved on the sheet: J1, J2, J3, J4, R1, R2, R3, R4
